File: esp32_battery_isolator.sch (KiCad schematic (older format))
At the start: 45 parts, among them J1 INPUT, J2 LOAD1, J3 BATT1, J4 BATT2, J5 LOAD2, J6 Conn_01x06_Female, J7 Conn_01x04_Female, Q1 BSC070N10LS5, Q2 BSC070N10LS5, Q3 BSC070N10LS5, Q4 BSC070N10LS5, SW1 TS-1102W-4316, U1 ME6119C33M5G, U2 ESP32-WROOM-32D, U3 ACS781LLRTR-050B, U4 ACS781LLRTR-050B, U5 ACS781LLRTR-050B, U6 ACS781LLRTR-050B, U7 LM75BDP,118

Commit message: Rev 1 Shipped to JLCPCB
Changed lines of the file:
@@
 Text GLabel 4820 6592 2    50   Output ~ 0
 AUX_1
-Text GLabel 3620 6292 0    50   Output ~ 0
+Text GLabel 4820 5692 2    50   Output ~ 0
 AUX_2
 Text GLabel 4820 6192 2    50   Output ~ 0
@@
 NoConn ~ 4820 6092
 NoConn ~ 4820 5792
-NoConn ~ 4820 5692
 NoConn ~ 4820 5392
 Text Notes 3396 1280 0    50   ~ 0
@@
 Text Notes 2090 7148 0    50   ~ 0
 Temp
+NoConn ~ 3620 6292
 $EndSCHEMATC

Commit message: WIP
Parts:
- removed J1: INPUT, Acea:AMASS_XT90-F_1x02_P11mm_Vertical, symbol Connector:Conn_01x02_Male
- removed U1: ME6119C33M5G, Package_TO_SOT_SMD:SOT-23-5, symbol Regulator_Linear:TLV70012_SOT23-5
- removed U3, U6: ACS781LLRTR-050B, Sensor_Current:Allegro_PSOF-7_4.8x6.4mm_P1.60mm, symbol Sensor_Current:ACS781xLRTR-050B
- added SW2: TS-1102W-4316, Button_Switch_SMD:SW_Push_1P1T_NO_6x6mm_H9.5mm, symbol MAX17260:TACT-SWITCH
- added U1: AMS1117-3.3, Package_TO_SOT_SMD:SOT-223-3_TabPin2, symbol Regulator_Linear:AMS1117-3.3
Connections:
- net labels added: RST
- net labels removed: LOAD_1_C, LOAD_2_C
- wire segments 72 -> 61
- no-connect marks 24 -> 23
Other:
- note added: "Batt 1 (MAIN)"
- note added: "Batt 2 (AUX)"
- note added: "SPARE ADC"
- note removed: "Aux Batt 1"
- note removed: "Aux Batt 2"
- note removed: "Input\n"
