File: esp32_battery_isolator.kicad_sch (KiCad schematic)
At the start: 80 parts, among them J1 BATT1, J2 Conn_01x04_Female, J3 USB_B_Micro, J4 BATT2, J5 LOAD1, J6 CHGR, J7 LOAD2, J8 LOAD3, J9 Conn_01x03_Male, Q1 MMBT3904, Q10 AONR21357, Q11 AONR21357, Q12 MMBT3904, Q13 MMBT3906, Q14 MMBT3906, Q15 MMBT3904, Q16 MMBT3906, Q17 MMBT3904, Q18 MMBT3906, Q19 MMBT3904, Q2 AONR21357, Q20 AONR21357, Q21 AONR21357, Q3 MMBT3904, Q4 AONR21357, Q5 MMBT3904, Q6 MMBT3904, Q7 MMBT3904, Q8 AONR21357, Q9 MMBT3904, SW1 C480325, SW2 C480325, U1 ESP32-WROOM-32D, U2 XL1509_SOP8, U3 ADC128D818, U4 CC6903SO-30A, U5 CH340N, U6 CC6903SO-30A

Commit message: wip
Parts:
- removed J1: BATT1, Acea:AMASS_XT60PW-M, symbol Connector:Conn_01x02_Male
- removed J2: Conn_01x04_Female, Connector_PinSocket_2.54mm:PinSocket_1x04_P2.54mm_Vertical, symbol Connector:Conn_01x04_Female
- removed J3: USB_B_Micro, Acea:USB_Micro_SHOU-HAN-MicroXNJ_C404969_Horizontal, symbol esp32_battery_isolator-rescue:USB_B_Micro-Connector
- removed J4: BATT2, Acea:AMASS_XT60PW-M, symbol Connector:Conn_01x02_Male
- removed J5: LOAD1, Acea:AMASS_XT60PW-F, symbol Connector:Conn_01x02_Male
- removed J6: CHGR, Acea:AMASS_XT60PW-M, symbol Connector:Conn_01x02_Male
- removed J7: LOAD2, Acea:AMASS_XT60PW-F, symbol Connector:Conn_01x02_Male
- removed J8: LOAD3, Acea:AMASS_XT60PW-F, symbol Connector:Conn_01x02_Male
- removed Q20, Q21, Q4: AONR21357, Acea:DFN-TRANS_AONR21321, symbol Transistor_FET:QM6015D
- removed R18, R21: 3.6k, Resistor_SMD:R_0603_1608Metric, symbol Device:R_Small
- removed R19, R24: 11k, Resistor_SMD:R_0603_1608Metric, symbol Device:R_Small
- removed U4, U6: CC6903SO-30A, Package_SO:SOP-8_3.9x4.9mm_P1.27mm, symbol esp32_battery_isolator-rescue:CC6903-30A-Sensor_Current
- added C11, C17, C18, C4, C5, C6: 100n, Capacitor_SMD:C_0603_1608Metric, symbol Device:C_Small
- added H1, H10, H2, H3, H4, H5, H9: Cable_Connection, Acea:Rivneut_M6_Via, symbol Mechanical:MountingHole_Pad
- added H11, H12, H7, H8: MountingHole, MountingHole:MountingHole_3.2mm_M3_Pad_Via, symbol Mechanical:MountingHole
- added J2: USB_C_Receptacle_USB2.0, Connector_USB:USB_C_Receptacle_HRO_TYPE-C-31-M-12, symbol hardware_nrf52840_pa_beacon_hat:USB_C_Receptacle_USB2.0-Connector
- added Q5, Q6, Q7: HSBA100P03, Acea:LFPAK56, symbol Transistor_FET:QM6015D
- added R10, R12, R16, R4, R5, R9: 4mR, Acea:RS1050Metric_Pad5.3x2.5mm, symbol Device:R_Small
- added R18, R19: 5.1k, Resistor_SMD:R_0402_1005Metric, symbol Device:R
- added U10, U2, U3, U4, U7, U9: INA219BxDCN, Package_TO_SOT_SMD:SOT-23-8, symbol Analog_ADC:INA219BxDCN
- BZ1: footprint Buzzer_Beeper:SMDBuzzer_C201046 -> Acea:SMDBuzzer_C201046
- Q4: renamed from Q11; value AONR21357 -> HSBA100P03; footprint Acea:DFN-TRANS_AONR21321 -> Acea:LFPAK56; lcsc_part_number C431196 -> C701057; package DFN 3x3 -> (none)
- R22: value 11k -> 4mR; footprint Resistor_SMD:R_0603_1608Metric -> Acea:RS1050Metric_Pad5.3x2.5mm; lcsc_part_number C25950 -> C481476; lcsc_url https://lcsc.com/product-detail/Chip-Resistor-Surface-Mount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 -> (none); package 0603 -> 10050
- R23: value 3.6k -> 4mR; footprint Resistor_SMD:R_0603_1608Metric -> Acea:RS1050Metric_Pad5.3x2.5mm; lcsc_part_number C22980 -> C481476; lcsc_url https://lcsc.com/product-detail/Chip-Resistor-Surface-Mount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 -> (none); package 0603 -> 10050
- renumbered C15 to C1, C9 to C10, C10 to C12, C4 to C13, C5 to C14, C6 to C15, C7 to C16, C12 to C2, C1 to C3, C2 to C7, C3 to C8, C8 to C9, D4 to D1, D5 to D2, D1 to D4, D2 to D5, D9 to D6, D8 to D7, J9 to J1, Q3 to Q10, Q14 to Q11, Q2 to Q12, Q19 to Q13, Q9 to Q14, Q17 to Q15, Q18 to Q16, Q7 to Q17, Q10 to Q18, Q15 to Q19, Q6 to Q2, Q16 to Q20, Q8 to Q21, Q13 to Q3, Q12 to Q8, Q5 to Q9, R5 to R1, R7 to R11, R32 to R14, R28 to R15, R3 to R2, R31 to R20, R30 to R21, R10 to R26, R11 to R27, R12 to R28, R13 to R29, R1 to R3, R8 to R6, R4 to R7, R6 to R8, U2 to U5, U5 to U6, U3 to U8
Connections:
- net +3V3: now also C11.1, C17.1, C18.1, C4.1, C5.1, C6.1, U10.4 (VS), U10.8 (A1), U2.4 (VS), U3.4 (VS), U3.7 (A0), U4.4 (VS), U7.4 (VS), U9.4 (VS), U9.7 (A0), U9.8 (A1)
- net 5V: now also J2.A4 (VBUS), J2.A9 (VBUS), J2.B4 (VBUS), J2.B9 (VBUS)
- net B1VM: now also H1.1, R4.2, R5.2, U2.1 (IN+)
- net COM: now also Q5.3 (S), Q7.3 (S), R10.2, R12.1, R9.1, U3.2 (IN-), U4.1 (IN+)
- net D: now also Q5.2 (D), Q6.2 (D), Q7.2 (D)
- net D+: now also J2.A6 (D+), J2.B6 (D+)
- net D-: now also J2.A7 (D-), J2.B7 (D-)
- net G: now also Q5.1 (G), Q6.1 (G), Q7.1 (G)
- net GND: now also C11.2, C17.2, C18.2, C4.2, C5.2, C6.2, H4.1, J2.A1 (GND), J2.A12 (GND), J2.B1 (GND), J2.B12 (GND), J2.S1 (SHIELD), R18.1, R19.1, U10.3 (GND), U10.7 (A0), U2.3 (GND), U2.7 (A0), U2.8 (A1), U3.3 (GND), U3.8 (A1), U4.3 (GND), U4.8 (A1), U7.3 (GND), U7.8 (A1), U9.3 (GND); no longer R22.2
- net LOAD1: now also H5.1, R16.2, U7.1 (IN+); no longer Q12.2 (D)
- net LOAD2: now also R23.2, H10.1, U10.1 (IN+); no longer Q21.2 (D)
- net LOAD3: now also R22.2, H9.1, U9.1 (IN+); no longer Q18.2 (D)
- net SCL: now also U10.5 (SCL), U2.5 (SCL), U3.5 (SCL), U4.5 (SCL), U7.5 (SCL), U7.7 (A0), U9.5 (SCL)
- net SDA: now also U10.6 (SDA), U2.6 (SDA), U3.6 (SDA), U4.6 (SDA), U4.7 (A0), U7.6 (SDA), U9.6 (SDA)
- net 3v3VD: no longer names the net of U8.12 (IN4)
- net B1C: no longer names the net of Q4.3 (S)
- net B1C: now also Q6.3 (S), R4.1, R5.1, U2.2 (IN-)
- net B1CVD: no longer names the net of U8.14 (IN2)
- net B1CVD: no longer R22.1
- net B2CM: no longer names the net of R23.1
- net B2CM: now also Q21.2 (D), U10.2 (IN-)
- net B2CVD: no longer names the net of U8.13 (IN3)
- net B2CVD: no longer R23.2
- new net: Q12.2 (D), R16.1, U7.2 (IN-)
- new net: Q18.2 (D), R22.1, U9.2 (IN-)
- new net: J2.A5 (CC1), R18.2
- new net: H3.1, R10.1, U4.2 (IN-)
- new net: J2.B5 (CC2), R19.2
- new net B2VM: H2.1, R12.2, R9.2, U3.1 (IN+)
- no-connect marks 24 -> 27
Other:
- note added: "100A max cont. 400A pulsed"
- note added: "10W Max."
- note added: "40A Max."
- note added: "5W Max."
- note added: "80A Max."
- note added: "ADDR:1000000"
- note added: "ADDR:1000001"
- note added: "ADDR:1000002"
- note added: "ADDR:1000003"
- note added: "ADDR:1000004"
- note added: "ADDR:1000005"
- note added: "B1CM"
- note added: "B2CM"
- note added: "Batt 1 Isolator (starter)"
- note added: "Batt 2 CM (aux)"
- note added: "Buttons"
- note added: "CHGR"
- note added: "DC-DC Buck 40V>3.3V@600mA"
- note added: "ESP-32 Microcontroller"
- note added: "FAN"
- note added: "Ground"
- note added: "I2C"
- note added: "Load 1 (30A Max.)"
- note added: "Load 2 (30A Max.)"
- note added: "Load 3 (lights- 30A Max.)"
- note added: "Solar Charger Input"
- note added: "USB-C"
- note removed: "12V FAN"
- note removed: "25A max."
- note removed: "2A max."
- note removed: "3.4V max."
- note removed: "ADCs"
- note removed: "Batt 1 current measurement"
- note removed: "Batt 1 isolator (starter)"
- note removed: "Batt 2 connection (auxiliary)"
- note removed: "Batt 2 current measurement"
- note removed: "CLRs?"
- note removed: "DC-DC Buck (40V to 3.3V 600mA)"
- note removed: "ESP-32"
- note removed: "I2C Port"
- note removed: "Load 1 (freezer)"
- note removed: "Load 2 (fridge)"
- note removed: "Load 3 (lights)"
- note removed: "USB"
- moved on the sheet: BZ1, C1, C10, C12, C13, C14, C15, C16, C2, C3, C7, C8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

Commit message: 1st pass complete
Parts:
- C8: value 220uF -> 100uF(220uF); footprint Capacitor_SMD:C_Elec_6.3x7.7 -> Capacitor_SMD:C_Elec_6.3x5.4; lcsc_part_number C371974 -> C696189
- D3, D6, D7: footprint Diode_SMD:D_SOD-123 -> Diode_SMD:D_SMC; lcsc_part_number C8598 -> C211777
- J2: footprint Connector_USB:USB_C_Receptacle_HRO_TYPE-C-31-M-12 -> Acea:USB_C_Receptacle_HRO_TYPE-C-31-M-12
- R18, R19: footprint Resistor_SMD:R_0402_1005Metric -> Resistor_SMD:R_0603_1608Metric
- SW1, SW2: value C480325 -> C620183; lcsc_part_number C480325 -> C620183
Other:
- note added: "Mounting Holes"
- moved on the sheet: H11, H12, H7, H8

Commit message: small schematic tweaks
Parts:
- Q11, Q16, Q20: lcsc_part_number https://datasheet.lcsc.com/lcsc/1811141238_Shikues-MMBT3906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 -> C111114
- U10, U2, U3, U4, U7, U9: lcsc_part_number (none) -> C2155693
Changed lines of the file:
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@@
       (effects (font (size 1.27 1.27) italic) (justify left) hide)
     )
-    (property "Datasheet" "C111114" (id 3) (at 237.998 68.58 0)
+    (property "Datasheet" "https://datasheet.lcsc.com/lcsc/1811141238_Shikues-MMBT3906_C111114.pdf" (id 3) (at 237.998 68.58 0)
       (effects (font (size 1.27 1.27)) (justify left) hide)
     )
-    (property "lcsc_part_number" "https://datasheet.lcsc.com/lcsc/1811141238_Shikues-MMBT3906_C111114.pdf" (id 4) (at 237.998 68.58 0)
+    (property "lcsc_part_number" "C111114" (id 4) (at 237.998 68.58 0)
       (effects (font (size 1.27 1.27)) hide)
     )
@@
       (effects (font (size 1.27 1.27) italic) (justify left) hide)
     )
-    (property "Datasheet" "C111114" (id 3) (at 347.091 68.834 0)
+    (property "Datasheet" "https://datasheet.lcsc.com/lcsc/1811141238_Shikues-MMBT3906_C111114.pdf" (id 3) (at 347.091 68.834 0)
       (effects (font (size 1.27 1.27)) (justify left) hide)
     )
-    (property "lcsc_part_number" "https://datasheet.lcsc.com/lcsc/1811141238_Shikues-MMBT3906_C111114.pdf" (id 4) (at 347.091 68.834 0)
+    (property "lcsc_part_number" "C111114" (id 4) (at 347.091 68.834 0)
       (effects (font (size 1.27 1.27)) hide)
     )
@@
       (effects (font (size 1.27 1.27) italic) (justify left) hide)
     )
-    (property "Datasheet" "C111114" (id 3) (at 330.581 133.223 0)
+    (property "Datasheet" "https://datasheet.lcsc.com/lcsc/1811141238_Shikues-MMBT3906_C111114.pdf" (id 3) (at 330.581 133.223 0)
       (effects (font (size 1.27 1.27)) (justify left) hide)
     )
-    (property "lcsc_part_number" "https://datasheet.lcsc.com/lcsc/1811141238_Shikues-MMBT3906_C111114.pdf" (id 4) (at 330.581 133.223 0)
+    (property "lcsc_part_number" "C111114" (id 4) (at 330.581 133.223 0)
       (effects (font (size 1.27 1.27)) hide)
     )
@@
     )
     (property "Datasheet" "http://www.ti.com/lit/ds/symlink/ina219.pdf" (id 3) (at 290.068 58.42 0)
+      (effects (font (size 1.27 1.27)) hide)
+    )
+    (property "lcsc_part_number" "C2155693" (id 4) (at 281.178 55.88 0)
       (effects (font (size 1.27 1.27)) hide)
     )
@@
       (effects (font (size 1.27 1.27)) hide)
     )
+    (property "lcsc_part_number" "C2155693" (id 4) (at 96.52 78.105 0)
+      (effects (font (size 1.27 1.27)) hide)
+    )
     (pin "1")
     (pin "2")
@@
       (effects (font (size 1.27 1.27)) hide)
     )
+    (property "lcsc_part_number" "C2155693" (id 4) (at 373.761 118.618 0)
+      (effects (font (size 1.27 1.27)) hide)
+    )
     (pin "1")
     (pin "2")
@@
       (effects (font (size 1.27 1.27)) hide)
     )
+    (property "lcsc_part_number" "C2155693" (id 4) (at 168.275 120.65 0)
+      (effects (font (size 1.27 1.27)) hide)
+    )
     (pin "1")
     (pin "2")
@@
     )
     (property "Datasheet" "http://www.ti.com/lit/ds/symlink/ina219.pdf" (id 3) (at 399.161 58.674 0)
+      (effects (font (size 1.27 1.27)) hide)
+    )
+    (property "lcsc_part_number" "C2155693" (id 4) (at 390.271 56.134 0)
       (effects (font (size 1.27 1.27)) hide)
     )
@@
       (effects (font (size 1.27 1.27)) hide)
     )
+    (property "lcsc_part_number" "C2155693" (id 4) (at 168.021 58.166 0)
+      (effects (font (size 1.27 1.27)) hide)
+    )

Commit message: WIP
Other:
- note added: "Inestigate the INA3221 for voltage and current monitoring"
Changed lines of the file:
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@@
     (effects (font (size 1.27 1.27)) (justify left bottom))
+  )
+  (text "Inestigate the INA3221 for voltage and current monitoring"
+    (at 94.615 -6.35 0)
+    (effects (font (size 5.08 5.08)) (justify left bottom))
   )
   (text "ESP-32 Microcontroller" (at 19.3294 160.782 0)

Commit message: Changed from push pull to independent pull up and pull down mosfets
Parts:
- removed Q10, Q19, Q2: MMBT3904, Package_TO_SOT_SMD:SOT-23, symbol Transistor_BJT:MMBT3904
- removed Q11, Q20, Q3: MMBT3906, Package_TO_SOT_SMD:SOT-23, symbol Transistor_BJT:MMBT3906
- added Q10, Q11, Q2: Q_PMOS_GSD, Package_TO_SOT_SMD:SOT-23, symbol Device:Q_PMOS_GSD
- added Q19, Q20, Q3: 2N7002, Package_TO_SOT_SMD:SOT-23, symbol Transistor_FET:2N7002
- added R13, R17, R24: 5k, Resistor_SMD:R_0603_1608Metric, symbol Device:R_Small
Connections:
- net B1ON: now also U1.12 (IO27), Q3.1 (G); no longer R1.1, U1.8 (IO32)
- net COM: now also Q10.2 (S), Q11.2 (S), Q2.2 (S), R13.2, R17.2, R24.2
- net D: no longer Q4.2 (D), Q5.2 (D)
- net G: now also Q2.3 (D), Q3.3 (D)
- net GND: now also Q19.2 (S), Q20.2 (S), Q3.2 (S)
- net L1ON: now also U1.23 (IO15), Q19.1 (G); no longer R15.1, U1.13 (IO14)
- net L2ON: now also U1.29 (IO5), Q20.1 (G); no longer R21.1, U1.16 (IO13)
- net at Q9.3 (C): now also Q10.1 (G), R17.1
- net at Q12.1 (G): now also Q10.3 (D), Q19.3 (D)
- net at Q1.3 (C): now also Q2.1 (G), R13.1
- net at Q17.3 (C): now also Q11.1 (G), R24.1
- net at Q21.1 (G): now also Q11.3 (D), Q20.3 (D)
- new net: Q4.2 (D), Q5.2 (D)
- new net B1OFF: R1.1, U1.8 (IO32)
- new net L1OFF: R15.1, U1.13 (IO14)
- new net L2OFF: R21.1, U1.16 (IO13)
- no-connect marks 27 -> 24
Other:
- moved on the sheet: BZ1, C1, C10, C11, C12, C13, C14, C15, C16, C17, C18, C2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

Commit message: More cleanup
Parts:
- added C19: 100uF(220uF), Capacitor_SMD:C_Elec_6.3x5.4, symbol Device:CP_Small
Connections:
- net COM: now also C19.1
- net D: now also Q4.2 (D), Q5.2 (D)
- net GND: now also C19.2
Other:
- moved on the sheet: C12, C4, C6, C7, C8, C9, D1, D2, D3, D4, D5, H1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
