File: lite/esp32_battery_isolator.kicad_pcb (KiCad board)
At the start: 2 copper layers, 67.8 x 59.3 mm, 70 parts, among them J1 BATT1, J2 Conn_01x04_Female, J3 USB_B_Micro, J4 BATT2, J5 LOAD1, J6 CHGR, J7 LOAD2, J8 LOAD3, Q1 MMBT3904, Q10 WSD20L120DN, Q2 WSD20L120DN, Q3 MMBT3904, Q4 WSD20L120DN, Q5 MMBT3904, Q6 WSD20L120DN, Q7 MMBT3904, Q8 WSD20L120DN, Q9 MMBT3904, SW1 KMR221GLFS, SW2 KMR221GLFS, SW3 KMR221GLFS, U1 ESP32-WROOM-32D, U2 LD1086D2T33TR, U3 ADC128D818, U4 CC6903SO-30A, U5 CH330N, U6 CC6903SO-30A

Commit message: Rev C - RC1
enclosure may need some adjusting. Will do a test print and update if needed.
Parts:
- removed Q1, Q3, Q5, Q7, Q9: MMBT3904, Package_TO_SOT_SMD:SOT-23
- R1, R4, R8, R9: value 10k -> 10k2
- moved R17 5.40 mm to (143.0, 117.2)
- moved R4 4.26 mm to (133.8, 99.5)
- moved R20 4.16 mm to (144.2, 108.3)
- moved C9 2.29 mm to (160.9, 88.9), turned to 270 degrees
- moved J2 2.20 mm to (158.7, 89.2)
- moved J3 1.20 mm to (171.7, 92.0)
- moved Q6 0.97 mm to (129.6, 103.7)
- moved C7 0.55 mm to (139.2, 129.6)
- moved C6 0.48 mm to (138.1, 126.4)
- moved R12 0.48 mm to (137.4, 130.9)
- moved C5 0.38 mm to (139.2, 123.8)
- moved C1 0.35 mm to (133.9, 86.8)
- moved R13 0.35 mm to (127.2, 130.9)
- moved C12 0.32 mm to (133.9, 83.2)
- moved U6 0.28 mm to (128.9, 110.8)
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Connections:
- Q10 pad 4: Net-(Q10-Pad4) -> L3ON
- Q2 pad 4: Net-(Q1-Pad3) -> L1ON
- Q4 pad 4: Net-(Q3-Pad3) -> B1ON
- Q6 pad 4: Net-(Q5-Pad3) -> B2ON
- Q8 pad 4: Net-(Q7-Pad3) -> L2ON
- R14 pad 2: Net-(Q3-Pad3) -> B1ON
- R15 pad 2: Net-(Q5-Pad3) -> B2ON
- R16 pad 2: Net-(Q1-Pad3) -> L1ON
- R17 pad 2: Net-(Q7-Pad3) -> L2ON
- R20 pad 2: Net-(Q10-Pad4) -> L3ON
- R4 pad 1: GND -> Net-(R4-Pad1)
- R4 pad 2: Net-(R4-Pad2) -> GND
- U1 pad 14: Net-(R4-Pad2) -> Net-(R4-Pad1)
Routing:
- net Net-(Q3-Pad3): track 44.7 -> 0.00 mm
- net B1ON: track 29.4 -> 71.8 mm
- net +3V3: track 223.5 -> 188.9 mm, vias 9 -> 8
- net L1ON: track 54.6 -> 68.5 mm
- net Net-(Q1-Pad3): track 10.9 -> 0.00 mm
- net B1CVD: track 96.4 -> 88.3 mm
- net B2ON: track 13.2 -> 19.8 mm
- net Net-(Q7-Pad3): track 6.15 -> 0.00 mm
- net Net-(Q10-Pad4): track 6.11 -> 0.00 mm
- net Net-(Q5-Pad3): track 6.10 -> 0.00 mm
- net GND: track 82.1 -> 76.2 mm, vias 87 -> 84
- net B2VM: track 136.3 -> 141.3 mm, vias 8 -> 5
- net D+: track 9.42 -> 14.2 mm
- net L2ON: track 26.5 -> 23.0 mm
- net SDA: track 95.1 -> 98.5 mm
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- added copper zone on F.Cu, net +3V3

Commit message: REV C off to JLCPCB
Parts:
- moved R13 8.40 mm to (135.7, 130.8)
- moved R11 3.81 mm to (112.4, 125.5)
- moved R10 3.30 mm to (111.2, 124.2)
- moved R14 2.50 mm to (110.5, 122.8)
- moved R19 0.89 mm to (115.3, 126.8)
- moved R18 0.62 mm to (116.5, 129.2)
Routing:
- net GND: track 76.2 -> 55.3 mm, vias 84 -> 81
- net B2CM: track 67.0 -> 50.8 mm
- net B2VD: track 23.7 -> 15.3 mm
- net B1VD: track 42.0 -> 46.1 mm
- net B1VM: track 27.8 -> 24.7 mm
- net B1ON: track 71.8 -> 69.6 mm
- net B1CVD: track 88.3 -> 89.4 mm
- net 3v3VD: track 44.6 -> 45.4 mm
- net +3V3: track 188.9 -> 189.5 mm
- net B2C: vias 27 -> 32
Other:
- board text added: "B1"
- board text added: "B2"
- board text added: "B3"
- board text added: "CHG"
- board text added: "L1"
- board text added: "L2"
- board text added: "L3"
- board text removed: "BAT3"
- board text removed: "CHGR"
- board text removed: "LD1"
- board text removed: "LD2"
- board text removed: "LD3"

Commit message: REV D WIP
Parts:
- C10, C9: footprint Capacitor_SMD:C_0603_1608Metric -> Capacitor_SMD:C_0805_2012Metric
- C2, C3: value CP_Small -> 22uF 35V
- R6, R7: value 2.2k -> 2.55K; footprint Resistor_SMD:R_0603_1608Metric -> LED_SMD:LED_0603_1608Metric
- SW1, SW2, SW3: value KMR221GLFS -> TS4450P; footprint Button_Switch_SMD:SW_Push_1P1T_NO_CK_KMR2 -> Acea:TS4550TP
- moved R1 9.27 mm to (121.3, 84.3)
- moved R8 4.25 mm to (121.3, 82.3)
- moved SW3 2.11 mm to (112.5, 93.8)
- moved SW1 1.73 mm to (111.1, 85.7)
- moved SW2 1.49 mm to (116.8, 85.7)
- moved C9 0.53 mm to (161.2, 89.3)
- moved C10 0.18 mm to (162.1, 79.8)
Routing:
- net RST: track 38.8 -> 50.2 mm
- net GND: track 55.3 -> 47.1 mm, vias 81 -> 79
- net BOOT: track 64.5 -> 58.3 mm
- net MODE: track 29.3 -> 35.3 mm
- net D+: track 14.2 -> 11.3 mm
- net B1CVD: track 89.4 -> 91.9 mm
- net B1ON: track 69.6 -> 67.7 mm
- net +3V3: track 189.5 -> 187.9 mm
- net D-: track 15.3 -> 14.6 mm
- net SCL: track 109.0 -> 109.6 mm

Commit message: REV D complete
Parts:
- added R25: 200R, Resistor_SMD:R_0603_1608Metric, F.Cu at (110.7, 125.5)
- added R26: 330R, Resistor_SMD:R_0603_1608Metric, F.Cu at (112.0, 125.5)
- C1, C10, C12, C5, C6, C9: footprint Capacitor_SMD:C_0805_2012Metric -> Capacitor_SMD:C_0603_1608Metric
- C11, C4, C7: footprint Capacitor_Tantalum_SMD:CP_EIA-3216-18_Kemet-A -> Capacitor_Tantalum_SMD:CP_EIA-3528-21_Kemet-B
- C2: value 22uF 35V -> 100n; footprint Capacitor_SMD:C_Elec_5x5.4 -> Capacitor_SMD:C_0603_1608Metric
- C3: value 22uF 35V -> 1uF; footprint Capacitor_SMD:C_Elec_5x5.4 -> Capacitor_Tantalum_SMD:CP_EIA-3528-21_Kemet-B
- D3: value B1 LED -> MAIN LED
- D4: value B2 LED -> MAIN LED
- J1, J4, J6: footprint Connector_AMASS:AMASS_XT60-F_1x02_P7.20mm_Vertical -> Acea:AMASS_XT60PW-M
- J3: footprint Acea:USB_Micro-B_XKB_4BH89_SMT -> Acea:USB_Micro_SHOU-HAN-MicroXNJ_C404969_Horizontal
- J5, J7, J8: footprint Connector_AMASS:AMASS_XT60-F_1x02_P7.20mm_Vertical -> Acea:AMASS_XT60PW-F
- Q10, Q2, Q4, Q6, Q8: value WSD20L120DN -> AP6679GH-HF; footprint Package_SO:PowerPAK_SO-8_Single -> Package_TO_SOT_SMD:TO-252-2
- R1, R19, R22, R24, R4, R8, R9: value 10k2 -> 11k
- R10, R12, R14, R15, R16, R17, R20: value 105k -> 200k
- R11, R13: value 20k -> 33k
- R18, R21, R23: value 30k9 -> 3.6k
- R2, R3, R5, R6, R7: value 2.55K -> 3.6k; footprint LED_SMD:LED_0603_1608Metric -> Resistor_SMD:R_0603_1608Metric
- SW1, SW2, SW3: value TS4450P -> C492887
- U2: value LD1086D2T33TR -> LM317AG-TN3-R
- moved R19 72.3 mm to (173.4, 83.8)
- moved R18 70.6 mm to (170.7, 83.8)
- moved J6 61.5 mm to (171.7, 95.2), turned to 270 degrees
- moved C6 53.4 mm to (164.2, 79.8), turned to 0 degrees
- moved SW3 50.1 mm to (161.1, 106.2), turned to 0 degrees
- moved R9 49.6 mm to (165.2, 105.0)
- moved U3 49.5 mm to (163.4, 83.3)
- moved C5 49.1 mm to (160.8, 79.8), turned to 0 degrees
- moved R11 48.2 mm to (116.7, 77.5), turned to 90 degrees
- moved R2 46.5 mm to (158.8, 99.5), turned to 270 degrees
- moved C7 46.4 mm to (159.7, 88.0), turned to 180 degrees
- moved C4 45.4 mm to (157.7, 82.5), turned to 270 degrees
- moved R14 44.2 mm to (125.7, 81.3), turned to 0 degrees
- moved R10 43.7 mm to (116.7, 80.8), turned to 90 degrees
- moved D1 42.7 mm to (156.1, 92.2), turned to 180 degrees
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Connections:
- Q10 pad 1: B2C -> L3ON
- Q10 pad 2: B2C -> LOAD3
- Q2 pad 1: B2C -> L1ON
- Q2 pad 2: B2C -> LOAD1
- Q4 pad 1: B1VM -> B1ON
- Q4 pad 2: B1VM -> B1C
- Q6 pad 1: B2C -> B2ON
- Q6 pad 2: B2C -> COM
- Q8 pad 1: B2C -> L2ON
- Q8 pad 2: B2C -> LOAD2
- R4 pad 1: Net-(R4-Pad1) -> GND
- R4 pad 2: GND -> Net-(R4-Pad2)
- R9 pad 1: +3V3 -> MODE
- R9 pad 2: MODE -> +3V3
- U1 pad 14: Net-(R4-Pad1) -> Net-(R4-Pad2)
- U2 pad 1: GND -> Net-(R25-Pad2)
Routing:
- net +3V3: track 187.9 -> 48.5 mm, vias 8 -> 39
- net SCL: track 109.6 -> 29.6 mm, vias 2 -> 0
- net B2CVD: track 6.06 -> 64.0 mm, vias 0 -> 2
- net SDA: track 98.5 -> 45.3 mm
- net B1ON: track 67.7 -> 19.4 mm, vias 2 -> 0
- net B2CM: track 50.8 -> 2.89 mm
- net BOOT: track 58.3 -> 13.3 mm, vias 2 -> 0
- net B2VD: track 15.3 -> 56.7 mm
- net 3v3VD: track 45.4 -> 7.08 mm
- net B1CVD: track 91.9 -> 54.0 mm, vias 0 -> 2
- net TXD: track 6.47 -> 35.2 mm, vias 0 -> 2
- net B1VM: track 24.7 -> 1.67 mm, vias 4 -> 16
- net RXD: track 10.8 -> 33.4 mm, vias 0 -> 2
- net L1ON: track 68.5 -> 46.5 mm
- net GND: track 47.1 -> 67.8 mm, vias 79 -> 61
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- added copper zone on In2.Cu, net +3V3
- added copper zone on In1.Cu, net GND
- removed copper zone on B.Cu, net +3V3
- removed copper zone on F.Cu, net +3V3
- removed copper zone on B.Cu, net B2VM
- removed copper zone on B.Cu, net GND
Other:
- outline, holes or cut-outs redrawn
- copper layers 2 -> 4
- board text added: "BATTERY ISOLATOR LITE REV.D ACEA QUIGG 02/20"
- board text removed: "3v3"
- board text removed: "BAT1"
- board text removed: "BAT2"
- board text removed: "BATTERY ISOLATOR LITE REV.C ACEA QUIGG 12/20"
- board text removed: "SCL"
- board text removed: "SDA"
