File: lite/esp32_battery_isolator.sch (KiCad schematic (older format))
At the start: 66 parts, among them J1 BATT1, J2 Conn_01x04_Female, J3 USB_B_Micro, J4 BATT2, J5 LOAD1, J6 CHGR, J7 LOAD2, J8 LOAD3, Q1 MMBT3904, Q10 WSD20L120DN, Q2 WSD20L120DN, Q3 MMBT3904, Q4 WSD20L120DN, Q5 MMBT3904, Q6 WSD20L120DN, Q7 MMBT3904, Q8 WSD20L120DN, Q9 MMBT3904, SW1 KMR221GLFS, SW2 KMR221GLFS, SW3 KMR221GLFS, U1 ESP32-WROOM-32D, U2 LD1086D2T33TR, U3 ADC128D818, U4 CC6903SO-30A, U5 CH330N, U6 CC6903SO-30A

Commit message: Rev C - RC1
enclosure may need some adjusting. Will do a test print and update if needed.
Parts:
- removed Q1, Q3, Q5, Q7, Q9: MMBT3904, Package_TO_SOT_SMD:SOT-23, symbol Transistor_BJT:MMBT3904
- R1, R4, R8, R9: value 10k -> 10k2; lcsc_part_number C15401 -> C705802; lcsc_url https://lcsc.com/product-detail/Chip-Resistor-Surface-Mount_UNI-ROYAL-Uniroyal-Elec-0603WAJ0103T5E_C15401.html -> https://lcsc.com/product-detail/Chip-Resistor-Surface-Mount_YAGEO-RT0603BRE0710K2L_C705802.html; mfr_part_number 0603WAJ0103T5E -> RT0603BRE0710K2L
Connections:
- net B1ON: now also Q4.4 (G), R14.2
- net B2ON: now also Q6.4 (G), R15.2
- net GND: now also R4.2; no longer R4.1
- net L1ON: now also Q2.4 (G), R16.2
- net L2ON: now also Q8.4 (G), R17.2
- net L3ON: now also Q10.4 (G), R20.2
- net at U1.14 (IO12): now also R4.1; no longer R4.2
Other:
- moved on the sheet: C11, C12, J1, J4, J5, J7, J8

Commit message: REV C off to JLCPCB
Other:
- moved on the sheet: C10
Changed lines of the file:
@@
 L Device:C_Small C10
 U 1 1 5F73731C
-P 9500 4200
-F 0 "C10" H 9300 4450 50  0000 L CNN
-F 1 "100n" H 9250 4350 50  0000 L CNN
-F 2 "Capacitor_SMD:C_0603_1608Metric" H 9500 4200 50  0001 C CNN
-F 3 "https://datasheet.lcsc.com/szlcsc/1910111742_YAGEO-AC0603KRX7R0BB104_C408909.pdf" H 9500 4200 50  0001 C CNN
-F 4 "C408909" H 9500 4200 50  0001 C CNN "lcsc_part_number"
-F 5 "https://lcsc.com/product-detail/Multilayer-Ceramic-Capacitors-MLCC-SMD-SMT_YAGEO-AC0603KRX7R0BB104_C408909.html" H 9500 4200 50  0001 C CNN "lcsc_url"
-F 6 "20" H 9500 4200 50  0001 C CNN "lcsc_min_qty"
-F 7 "AC0603KRX7R0BB104" H 9500 4200 50  0001 C CNN "mfr_part_number"
-F 8 "0603" H 9500 4200 50  0001 C CNN "package"
-	1    9500 4200
+P 9500 4250
+F 0 "C10" H 9250 4250 50  0000 L CNN
+F 1 "100n" H 9250 4150 50  0000 L CNN
+F 2 "Capacitor_SMD:C_0603_1608Metric" H 9500 4250 50  0001 C CNN
+F 3 "https://datasheet.lcsc.com/szlcsc/1910111742_YAGEO-AC0603KRX7R0BB104_C408909.pdf" H 9500 4250 50  0001 C CNN
+F 4 "C408909" H 9500 4250 50  0001 C CNN "lcsc_part_number"
+F 5 "https://lcsc.com/product-detail/Multilayer-Ceramic-Capacitors-MLCC-SMD-SMT_YAGEO-AC0603KRX7R0BB104_C408909.html" H 9500 4250 50  0001 C CNN "lcsc_url"
+F 6 "20" H 9500 4250 50  0001 C CNN "lcsc_min_qty"
+F 7 "AC0603KRX7R0BB104" H 9500 4250 50  0001 C CNN "mfr_part_number"
+F 8 "0603" H 9500 4250 50  0001 C CNN "package"
+	1    9500 4250
 	1    0    0    -1
 $EndComp
@@
 L MAX17260:GND #PWR038
 U 1 1 5F737323
-P 9500 4300
-F 0 "#PWR038" H 9500 4300 30  0001 C CNN
-F 1 "GND" H 9500 4230 30  0001 C CNN
-F 2 "" H 9500 4300 60  0000 C CNN
-F 3 "" H 9500 4300 60  0000 C CNN
-	1    9500 4300
+P 9500 4350
+F 0 "#PWR038" H 9500 4350 30  0001 C CNN
+F 1 "GND" H 9500 4280 30  0001 C CNN
+F 2 "" H 9500 4350 60  0000 C CNN
+F 3 "" H 9500 4350 60  0000 C CNN
+	1    9500 4350
 	1    0    0    -1
 $EndComp
@@
 L power:+3V3 #PWR039
 U 1 1 5F77B761
-P 9600 4050
-F 0 "#PWR039" H 9600 3900 50  0001 C CNN
-F 1 "+3V3" H 9615 4223 50  0000 C CNN
-F 2 "" H 9600 4050 50  0001 C CNN
-F 3 "" H 9600 4050 50  0001 C CNN
-	1    9600 4050
-	1    0    0    -1
-$EndComp
-Wire Wire Line
-	9200 4350 9200 4100
-Wire Wire Line
-	9200 4100 9500 4100
-Wire Wire Line
-	9500 4100 9600 4100
-Wire Wire Line
-	9600 4100 9600 4050
-Connection ~ 9500 4100
+P 9200 4100
+F 0 "#PWR039" H 9200 3950 50  0001 C CNN
+F 1 "+3V3" H 9215 4273 50  0000 C CNN
+F 2 "" H 9200 4100 50  0001 C CNN
+F 3 "" H 9200 4100 50  0001 C CNN
+	1    9200 4100
+	1    0    0    -1
+$EndComp
+Wire Wire Line
+	9200 4350 9200 4150
 NoConn ~ 9600 4850
 $Comp
@@
 Wire Wire Line
 	2800 4900 3050 4900
+Wire Wire Line
+	9500 4150 9200 4150
+Connection ~ 9200 4150
+Wire Wire Line
+	9200 4150 9200 4100
 $EndSCHEMATC

Commit message: REV D WIP
Parts:
- C10, C9: footprint Capacitor_SMD:C_0603_1608Metric -> Capacitor_SMD:C_0805_2012Metric; lcsc_min_qty 20 -> 100; lcsc_part_number C408909 -> C128353; lcsc_url https://lcsc.com/product-detail/Multilayer-Ceramic-Capacitors-MLCC-SMD-SMT_YAGEO-AC0603KRX7R0BB104_C408909.html -> https://lcsc.com/product-detail/Multilayer-Ceramic-Capacitors-MLCC-SMD-SMT_Walsin-Tech-Corp-0805B104K250_C128353.html; mfr_part_number AC0603KRX7R0BB104 -> 0805B104K250; package 0603 -> 0805
- C2, C3: value CP_Small -> 22uF 35V
- R6, R7: value 2.2k -> 2.55K; footprint Resistor_SMD:R_0603_1608Metric -> LED_SMD:LED_0603_1608Metric; lcsc_min_qty 100 -> 50; lcsc_part_number C384262 -> C304726; lcsc_url https://lcsc.com/product-detail/Chip-Resistor-Surface-Mount_Walsin-Tech-Corp-Walsin-Tech-Corp-2-2KR-222-5_C384262.html -> https://lcsc.com/product-detail/Chip-Resistor-Surface-Mount_FH-Guangdong-Fenghua-Advanced-Tech-RS-03K2551FT_C304726.html; mfr_part_number WR06X222 JTL -> RS-03K2551FT
- SW1, SW2, SW3: value KMR221GLFS -> TS4450P; footprint Button_Switch_SMD:SW_Push_1P1T_NO_CK_KMR2 -> Acea:TS4550TP; lcsc_min_qty 1 -> 50; lcsc_part_number C72443 -> C412373; lcsc_url https://lcsc.com/product-detail/Tactile-Switches_C-K_KMR221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 -> https://lcsc.com/product-detail/Tactile-Switches_SHOU-HAN-T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; mfr_part_number KMR221GLFS -> TS4550TP; package KMR2 -> 4.5mm,4.5mm SMD
- U3: mfr_part_number https://lcsc.com/product-detail/Analog-To-Digital-Converter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 -> ADC128D818CIMTX

Commit message: REV D complete
Parts:
- removed Q10, Q2, Q6, Q8: WSD20L120DN, Package_SO:PowerPAK_SO-8_Single, symbol Transistor_FET:Si7141DP
- removed U2: LD1086D2T33TR, Package_TO_SOT_SMD:TO-252-2, symbol Regulator_Linear:LD1086D2T33TR
- added Q10, Q2, Q6, Q8: AP6679GH-HF, Package_TO_SOT_SMD:TO-252-2, symbol Transistor_FET:QM6015D
- added R25: 200R, Resistor_SMD:R_0603_1608Metric, symbol Device:R_Small
- added R26: 330R, Resistor_SMD:R_0603_1608Metric, symbol Device:R_Small
- added U2: LM317AG-TN3-R, Package_TO_SOT_SMD:TO-252-2, symbol Regulator_Linear:LM317_TO-252
- C1, C10, C12, C5, C6, C9: footprint Capacitor_SMD:C_0805_2012Metric -> Capacitor_SMD:C_0603_1608Metric; lcsc_min_qty 100 -> (none); lcsc_part_number C128353 -> C14663; lcsc_url https://lcsc.com/product-detail/Multilayer-Ceramic-Capacitors-MLCC-SMD-SMT_Walsin-Tech-Corp-0805B104K250_C128353.html -> https://lcsc.com/product-detail/Multilayer-Ceramic-Capacitors-MLCC-SMD-SMT_100nF-104-10-50V_C14663.html/?href=jlc-SMT; mfr_part_number 0805B104K250 -> (none); package 0805 -> 0603
- C11, C4, C7: footprint Capacitor_Tantalum_SMD:CP_EIA-3216-18_Kemet-A -> Capacitor_Tantalum_SMD:CP_EIA-3528-21_Kemet-B; lcsc_min_qty 5 -> (none); lcsc_part_number C126949 -> C169224; lcsc_url https://lcsc.com/product-detail/Tantalum-Capacitors_Hunan-X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 -> (none); mfr_part_number CA45-A035K105T -> (none); package CASE_A_3216 -> CASE-B_3528
- C2: value 22uF 35V -> 100n; footprint Capacitor_SMD:C_Elec_5x5.4 -> Capacitor_SMD:C_0603_1608Metric; symbol Device:CP_Small -> Device:C_Small; lcsc_min_qty 20 -> (none); lcsc_part_number C23289 -> C14663; lcsc_url https://lcsc.com/product-detail/Aluminum-Electrolytic-Capac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 -> https://lcsc.com/product-detail/Multilayer-Ceramic-Capacito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; mfr_part_number RVT1V220M0505 -> (none); package 5x5.4 -> 0603
- C3: value 22uF 35V -> 1uF; footprint Capacitor_SMD:C_Elec_5x5.4 -> Capacitor_Tantalum_SMD:CP_EIA-3528-21_Kemet-B; lcsc_min_qty 20 -> (none); lcsc_part_number C23289 -> C169224; lcsc_url https://lcsc.com/product-detail/Aluminum-Electrolytic-Capac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 -> (none); mfr_part_number RVT1V220M0505 -> (none); package 5x5.4 -> CASE-B_3528
- D1: lcsc_min_qty 20 -> (none); lcsc_part_number C72044 -> C2286; lcsc_url https://lcsc.com/product-detail/Light-Emitting-Diodes-LED_0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 -> https://jlcpcb.com/parts/componentSearch?secondSortUuid=ac4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; mfr_part_number 19-217/R6C-AL1M2VY/3T -> (none)
- D2: lcsc_min_qty 50 -> (none)
- D3: value B1 LED -> MAIN LED; lcsc_min_qty 20 -> (none); lcsc_part_number C72044 -> C2286; lcsc_url https://lcsc.com/product-detail/Light-Emitting-Diodes-LED_0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 -> https://jlcpcb.com/parts/componentSearch?secondSortUuid=ac4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; mfr_part_number 19-217/R6C-AL1M2VY/3T -> (none)
- D4: value B2 LED -> MAIN LED; lcsc_min_qty 20 -> (none); lcsc_part_number C72044 -> C2286; lcsc_url https://lcsc.com/product-detail/Light-Emitting-Diodes-LED_0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 -> https://jlcpcb.com/parts/componentSearch?secondSortUuid=ac4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; mfr_part_number 19-217/R6C-AL1M2VY/3T -> (none)
- J1, J4, J6: footprint Connector_AMASS:AMASS_XT60-F_1x02_P7.20mm_Vertical -> Acea:AMASS_XT60PW-M; lcsc_part_number (none) -> C98732; other_URL https://www.frontlinehobbies.com.au/g-force-xt60-gold-conne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 -> (none)
- J3: footprint Acea:USB_Micro-B_XKB_4BH89_SMT -> Acea:USB_Micro_SHOU-HAN-MicroXNJ_C404969_Horizontal; lcsc_min_qty 10 -> (none); lcsc_part_number C319172 -> C404969; lcsc_url https://lcsc.com/product-detail/USB-Connectors_XKB-Enterpri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 -> https://lcsc.com/product-detail/USB-Connectors_SHOU-HAN-Mic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; mfr_part_number U253-051T-4BH89-F1B -> (none)
- J5, J7, J8: footprint Connector_AMASS:AMASS_XT60-F_1x02_P7.20mm_Vertical -> Acea:AMASS_XT60PW-F; lcsc_part_number (none) -> C428722; other_URL https://www.frontlinehobbies.com.au/g-force-xt60-gold-conne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 -> (none)
- Q4: value WSD20L120DN -> AP6679GH-HF; footprint Package_SO:PowerPAK_SO-8_Single -> Package_TO_SOT_SMD:TO-252-2; symbol Transistor_FET:Si7141DP -> Transistor_FET:QM6015D; lcsc_min_qty 1 -> (none); lcsc_part_number C148395 -> C124530; lcsc_url https://lcsc.com/product-detail/MOSFET_Winsok-Semicon-WSD20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 -> https://lcsc.com/product-detail/MOSFET_Advanced-Power-Elec-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; mfr_part_number WSD20L120DN -> (none); package SON8 -> TO-252-2
- R1, R19, R22, R24, R4, R8, R9: value 10k2 -> 11k; lcsc_min_qty 100 -> (none); lcsc_part_number C705802 -> C25950; lcsc_url https://lcsc.com/product-detail/Chip-Resistor-Surface-Mount_YAGEO-RT0603BRE0710K2L_C705802.html -> https://lcsc.com/product-detail/Chip-Resistor-Surface-Mount_Uniroyal-Elec-0603WAF1102T5E_C25950.html/?href=jlc-SMT; mfr_part_number RT0603BRE0710K2L -> (none)
- R10, R12, R14, R15, R16, R17, R20: value 105k -> 200k; lcsc_min_qty 5 -> (none); lcsc_part_number C491109 -> C25811; lcsc_url https://lcsc.com/product-detail/New-Arrivals_PANASONIC-ERA3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 -> https://lcsc.com/product-detail/Chip-Resistor-Surface-Mount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; mfr_part_number ERA3AEB1053V -> (none)
- R11, R13: value 20k -> 33k; lcsc_min_qty 20 -> (none); lcsc_part_number C319766 -> C4216; lcsc_url https://lcsc.com/product-detail/Others_Viking-Tech-AR03BTCX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 -> https://lcsc.com/product-detail/Chip-Resistor-Surface-Mount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; mfr_part_number AR03BTCX2002 -> (none)
- R18, R21, R23: value 30k9 -> 3.6k; lcsc_min_qty 100 -> (none); lcsc_part_number C23022 -> C22980; lcsc_url https://lcsc.com/product-detail/Chip-Resistor-Surface-Mount_UNI-ROYAL-Uniroyal-Elec-0603WAF3092T5E_C23022.html -> https://lcsc.com/product-detail/Chip-Resistor-Surface-Mount_Uniroyal-Elec-0603WAF3601T5E_C22980.html/?href=jlc-SMT; mfr_part_number 0603WAF3092T5E -> (none)
- R2, R3, R5, R6, R7: value 2.55K -> 3.6k; footprint LED_SMD:LED_0603_1608Metric -> Resistor_SMD:R_0603_1608Metric; lcsc_min_qty 50 -> (none); lcsc_part_number C304726 -> C22980; lcsc_url https://lcsc.com/product-detail/Chip-Resistor-Surface-Mount_FH-Guangdong-Fenghua-Advanced-Tech-RS-03K2551FT_C304726.html -> https://lcsc.com/product-detail/Chip-Resistor-Surface-Mount_Uniroyal-Elec-0603WAF3601T5E_C22980.html/?href=jlc-SMT; mfr_part_number RS-03K2551FT -> (none)
- SW1, SW2, SW3: value TS4450P -> C492887; lcsc_min_qty 50 -> (none); lcsc_part_number C412373 -> C492887; lcsc_url https://lcsc.com/product-detail/Tactile-Switches_SHOU-HAN-T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 -> (none); mfr_part_number TS4550TP -> TS-1091S-A5B3-C1D2
Connections:
- net +3V3: now also R9.2, R25.1, U2.2 (VO); no longer R9.1
- net B1C: now also Q4.2 (D); no longer Q4.5 (D)
- net B1ON: now also Q4.1 (G); no longer Q4.4 (G)
- net B1VM: no longer Q4.1 (S), Q4.2 (S)
- net B2C: now also Q10.3 (S), Q2.3 (S), Q6.3 (S), Q8.3 (S)
- net B2ON: now also Q6.1 (G)
- net B2VM: now also U2.3 (VI)
- net COM: now also Q6.2 (D)
- net GND: now also R4.1, R26.2; no longer R4.2
- net L1ON: now also Q2.1 (G)
- net L2ON: now also Q8.1 (G)
- net L3ON: now also Q10.1 (G)
- net LOAD1: now also Q2.2 (D)
- net LOAD2: now also Q8.2 (D)
- net LOAD3: now also Q10.2 (D)
- net MODE: now also R9.1; no longer R9.2
- net at U1.14 (IO12): now also R4.2; no longer R4.1
- new net: R25.2, R26.1, U2.1 (ADJ)
Other:
- moved on the sheet: C3, D1, D2
